File: schematics/sch/GroundStationCR.sch (EAGLE design)
At the start: 13 parts

Commit message: minor fixes
Parts:
- removed C4, C5: (no value), resistor:C-EU050-025X075
- removed CON_HIGH, CON_LOW: (no value), pinhead:PINHD-1X6
- added B1: SPARKFUN_LOGIC_LEVEL_CONVERTER, sparkfun-boards:SPARKFUN_LOGIC_LEVEL_CONVERTER
- added C6: 10uF, resistor:C-EU050-025X075
- added C7: 100nF, resistor:C-EU050-025X075
- added D1: 1N5908, diode:1N5908
- added D2: CLEAR, sparkfun-led:LED-RGB-CACLEAR
- added J2: POWER_JACKPTH_LOCK, sparkfun-connectors:POWER_JACKPTH_LOCK
- added LED1, LED2: (no value), led:LED3MM
- added R1, R2: 10k, rcl:R-EU_0207/7
- added R3, R4, R5, R6, R7: 500R, rcl:R-EU_0207/7
- added R8: (no value), rcl:R-EU_0207/5V
- C1, C2, C3: value (none) -> 100nF
- MICROSD: device pinhead:PINHD-1X9 -> pinhead:PINHD-1X8
Connections:
- removed net CS: CON_HIGH.1, U$1.D10
- removed net CS_L: CON_LOW.6, MICROSD.4
- removed net RS: U$1.D4, U$3.1
- removed net SCLK: CON_HIGH.2, U$1.D13
- removed net SCLK_L: CON_LOW.5, MICROSD.5, U$3.4
- new net B: R6.1, U$1.D5
- new net CS_R: B1.HV_TXO_2, U$1.D8
- new net CS_R_L: B1.LV_TXI_2, U$3.1
- new net CS_S: MICROSD.4, U$1.D9
- new net G: R5.1, U$1.D6
- new net INT_R: U$1.D2, U$2.4
- new net N$1: D1.A, J2.PWR
- new net N$4: R1.1, R2.2, U$1.A1
- new net N$5: LED1.C, R3.2
- new net N$6: LED2.C, R4.2
- new net N$7: D2.GRN, R5.2
- new net N$8: D2.BLU, R6.2
- new net N$9: D2.RED, R7.2
- new net R: R7.1, U$1.D7
- new net SCK: B1.HV_RXI_2, MICROSD.6, U$1.D13
- new net SCK_L: B1.LV_RXO_2, U$3.4
- net +5V: now also B1.HV, C3.2, D2.A, MICROSD.1, TERMOMETER.2; no longer C4.1, CON_HIGH.4, TERMOMETER.1
- net 3.3V: now also B1.LV, C7.1, LED2.A, U$1.A0; no longer C3.1, C5.2, CON_LOW.3, MICROSD.9
- net GND: now also B1.GND, B1.GND@2, C3.1, C6.2, C7.2, J2.GND, J2.GNDBREAK, MICROSD.3, R2.1, R3.1, R4.1; no longer C3.2, C4.2, C5.1, CON_HIGH.3, CON_LOW.4, MICROSD.8
- net MISO: now also B1.HV_TXO_1, MICROSD.7, R8.1, R8.2; no longer CON_HIGH.6
- net MISO_L: now also B1.LV_TXI_1; no longer CON_LOW.1, MICROSD.7
- net MOSI: now also B1.HV_RXI_1, MICROSD.5; no longer CON_HIGH.5
- net MOSI_L: now also B1.LV_RXO_1; no longer CON_LOW.2, MICROSD.6
- net VIN: now also C6.1, D1.C, LED1.A, R1.2
Other:
- note added: "LED Debug"
- note added: "Zasilanie"
- moved on the sheet: C2, C3, DCCONVERTER, U$2
