File: schematics/brd/cansat.brd (EAGLE design)
At the start: 65.7 x 36.2 mm, 27 parts

Commit message: optocoupler on radio/gps vcc
Parts:
- added OK1: LTV816, optocoupler:DIL04
- added R5: 400R, eagle-ltspice:R1206
- added SJ3: (no value), jumper:SJ
Connections:
- removed net GND@5: RASPIZERO.20
- removed net GND@6: RASPIZERO.30
- removed net GND@7: RASPIZERO.34
- removed net GND@8: RASPIZERO.6
- new net N$2: OK1.1, R5.2
- new net VCC_OPTO: C2.2, C4.1, GPS.2, OK1.3, RADIOR.2, SJ3.1
- net 3.3V: now also OK1.4, SJ3.2; no longer C2.2, C4.1, GPS.2, RADIOR.2
- net EX1: now also R5.1
- net GND: now also OK1.2, RASPIZERO.20, RASPIZERO.30, RASPIZERO.34, RASPIZERO.6
- net R_INT: now also RASPIZERO.35
Routing:
- net GND: track 104.9 -> 168.4 mm
- net VCC_OPTO: track 0.00 -> 48.6 mm, vias 0 -> 4
- net EX1: track 0.00 -> 42.9 mm, vias 0 -> 3
- net R_INT: track 0.00 -> 35.6 mm
- net ENCODER2_DIR: track 60.6 -> 57.2 mm
- net 3.3V: track 130.2 -> 133.2 mm
- net N$2: track 0.00 -> 2.33 mm
- net ENCODER2_ADC: track 31.9 -> 33.0 mm
- net RS: track 19.4 -> 18.5 mm
- net SDA: track 76.8 -> 76.0 mm
